File: Hardware/Inverter.kicad_sch (KiCad schematic)
At the start: 56 parts, among them J2 Conn_01x02, J3 Conn_01x02, J4 Conn_01x01, J5 Conn_01x01, J6 Conn_01x01, Q1 CSD18532NQ5B, Q2 CSD18532NQ5B, Q3 CSD18532NQ5B, Q4 CSD18532NQ5B, Q5 CSD18532NQ5B, Q6 CSD18532NQ5B, U4 INA240A1PW, U5 LM321, U6 INA240A1PW, U7 INA240A1PW

Commit message: update BOM
Parts:
- Q1, Q2, Q3, Q4, Q5, Q6: value CSD18532NQ5B -> WSD30100DN56; LCSC Part # C2862136 -> C148393
Changed lines of the file:
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@@
 			)
 		)
-		(property "Value" "CSD18532NQ5B"
+		(property "Value" "WSD30100DN56"
 			(at 88.9 157.4799 0)
 			(show_name no)
@@
 			)
 		)
-		(property "Datasheet" "http://www.ti.com/lit/gpn/csd18532nq5b"
+		(property "Datasheet" ""
 			(at 87.63 160.02 0)
 			(hide yes)
@@
 			)
 		)
-		(property "LCSC Part #" "C2862136"
+		(property "LCSC Part #" "C148393"
 			(at 82.55 156.21 0)
 			(hide yes)
@@
 			)
 		)
-		(property "Value" "CSD18532NQ5B"
+		(property "Value" "WSD30100DN56"
 			(at 88.9 99.0599 0)
 			(show_name no)
@@
 			)
 		)
-		(property "Datasheet" "http://www.ti.com/lit/gpn/csd18532nq5b"
+		(property "Datasheet" ""
 			(at 87.63 101.6 0)
 			(hide yes)
@@
 			)
 		)
-		(property "LCSC Part #" "C2862136"
+		(property "LCSC Part #" "C148393"
 			(at 82.55 97.79 0)
 			(hide yes)
@@
 			)
 		)
-		(property "Value" "CSD18532NQ5B"
+		(property "Value" "WSD30100DN56"
 			(at 88.9 115.5699 0)
 			(show_name no)
@@
 			)
 		)
-		(property "Datasheet" "http://www.ti.com/lit/gpn/csd18532nq5b"
+		(property "Datasheet" ""
 			(at 87.63 118.11 0)
 			(hide yes)
@@
 			)
 		)
-		(property "LCSC Part #" "C2862136"
+		(property "LCSC Part #" "C148393"
 			(at 82.55 114.3 0)
 			(hide yes)
@@
 			)
 		)
-		(property "Value" "CSD18532NQ5B"
+		(property "Value" "WSD30100DN56"
 			(at 88.9 57.1499 0)
 			(show_name no)
@@
 			)
 		)
-		(property "Datasheet" "http://www.ti.com/lit/gpn/csd18532nq5b"
+		(property "Datasheet" ""
 			(at 87.63 59.69 0)
 			(hide yes)
@@
 			)
 		)
-		(property "LCSC Part #" "C2862136"
+		(property "LCSC Part #" "C148393"
 			(at 82.55 55.88 0)
 			(hide yes)
@@
 			)
 		)
-		(property "Value" "CSD18532NQ5B"
+		(property "Value" "WSD30100DN56"
 			(at 88.9 40.6399 0)
 			(show_name no)
@@
 			)
 		)
-		(property "Datasheet" "http://www.ti.com/lit/gpn/csd18532nq5b"
+		(property "Datasheet" ""
 			(at 87.63 43.18 0)
 			(hide yes)
@@
 			)
 		)
-		(property "LCSC Part #" "C2862136"
+		(property "LCSC Part #" "C148393"
 			(at 82.55 39.37 0)
 			(hide yes)
@@
 			)
 		)
-		(property "Value" "CSD18532NQ5B"
+		(property "Value" "WSD30100DN56"
 			(at 88.9 173.9899 0)
 			(show_name no)
@@
 			)
 		)
-		(property "Datasheet" "http://www.ti.com/lit/gpn/csd18532nq5b"
+		(property "Datasheet" ""
 			(at 87.63 176.53 0)
 			(hide yes)
@@
 			)
 		)
-		(property "LCSC Part #" "C2862136"
+		(property "LCSC Part #" "C148393"
 			(at 82.55 172.72 0)
 			(hide yes)
