File: Hardware/foc_driver.kicad_pcb (KiCad board)
At the start: 2 copper layers, 60 x 56 mm, 132 parts, among them J1 Conn_01x03_MountingPin, J10 Conn_01x06_MountingPin, J11 Conn_01x05_MountingPin, J2 Conn_01x02, J3 Conn_01x02, J4 Conn_01x01, J5 Conn_01x01, J6 Conn_01x01, J7 USB_C_Receptacle_USB2.0_16P, J8 Conn_01x03_MountingPin, J9 Conn_01x03_MountingPin, Q1 CSD18532NQ5B, Q2 CSD18532NQ5B, Q3 CSD18532NQ5B, Q4 CSD18532NQ5B, Q5 CSD18532NQ5B, Q6 CSD18532NQ5B, U1 STM32F405RGTx, U10 AS5047D, U2 DRV8323RHRGZR, U3 LP2985-3.3, U4 INA240A1PW, U5 LM321, U6 INA240A1PW, U7 INA240A1PW, U8 USBLC6-2SC6, U9 TJA1051TK-3, Y1 12MHz

Commit message: update BOM
Parts:
- Q1, Q2, Q3, Q4, Q5, Q6: value CSD18532NQ5B -> WSD30100DN56
